Commit message: normalement c'est ok

File: socle.urdf (robot description, URDF)
Before this commit: robot socle, 1 links, 0 joints
Links:
- link socle: mass 1 -> None; geometry visual mesh filename=package://socle stl.stl scale=0.001 0.001 0.001

Commit message: collision socle

File: socle.urdf (robot description, URDF)
Before this commit: robot socle, 1 links, 0 joints
Links:
- link socle: geometry collision mesh filename=package://socle stl.stl scale=0.001 0.001 0.001; visual mesh filename=package://socle stl.stl scale=0.001 0.001 0.001
