Commit message: ajout de la gravité et collision du cube

File: cube.urdf (robot description, URDF)
Before this commit: robot cube, 1 links, 0 joints
Links:
- link cube: geometry collision box size=0.06 0.06 0.06; visual box size=0.06 0.06 0.06

Commit message: collision test

File: cube.urdf (robot description, URDF)
Before this commit: robot cube, 1 links, 0 joints
Links:
- link cube: geometry collision box size=0.03 0.03 0.03; visual box size=0.03 0.03 0.03
